File: MultiMacro.kicad_sch (KiCad schematic)
At the start: 35 parts, among them J1 Conn_01x02, SW1 SW_Push, SW10 SW_Push, SW12 SW_Push, SW13 SW_Push, SW14 SW_Push, SW15 SW_Push, SW16 SW_Push, SW2 SW_Push, SW2 SW_SPDT_312, SW3 SW_Push, SW4 SW_Push, SW5 SW_Push, SW6 SW_Push, SW7 SW_Push, SW8 SW_Push, SW9 SW_Push, U1 SuperMini nRF52840, U10 XL-3528RGBC-WS2812B, U11 XL-3528RGBC-WS2812B, U12 XL-3528RGBC-WS2812B, U13 XL-3528RGBC-WS2812B, U14 XL-3528RGBC-WS2812B, U2 XL-3528RGBC-WS2812B, U3 XL-3528RGBC-WS2812B, U4 XL-3528RGBC-WS2812B, U5 XL-3528RGBC-WS2812B, U6 XL-3528RGBC-WS2812B, U7 XL-3528RGBC-WS2812B, U8 XL-3528RGBC-WS2812B, U9 XL-3528RGBC-WS2812B

Commit message: chore: Update license info in schematics
Other:
- title: (none) -> Mutenix Macroboard
Changed lines of the file:
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@@
 	(generator_version "8.0")
 	(paper "A4")
+	(title_block
+		(title "Mutenix Macroboard")
+		(date "2025-01-27")
+		(rev "V1.0")
+		(comment 1 "SPDX-License-Info: CERN-OHL-S-2.0 license")
+		(comment 2 "Author: Matthias Bilger <matthias@bilger.info>")
+	)
 	(junction
 		(at 160.02 116.84)
